File: MiSTeX-Pmod/MiSTeX-Pmod.kicad_sch (KiCad schematic)
At the start: 29 parts, among them CN1 NASB0-S6701-TS50, CN2 NASB0-S6701-TS50, J1 Pmod, J2 USB_A, J3 Conn_01x03_Male, J4 Pmod, J5 Connector_USB_C_Receptacle_US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, SW1 TS-1187A-B-A-B

Commit message: change USB host connector, old one was out of stock
Parts:
- J2: footprint easyeda2kicad:USB-A-SMD_USB-302S -> easyeda2kicad:USB-A-SMD_GT-USB-2004-CWG1A; LCSC C112455 -> C5117890
Changed lines of the file:
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@@
   (symbol (lib_id "power:GND") (at 112.903 111.506 0) (unit 1)
     (in_bom yes) (on_board yes) (fields_autoplaced)
-    (property "Reference" "#PWR?" (id 0) (at 112.903 117.856 0)
+    (property "Reference" "#PWR0101" (id 0) (at 112.903 117.856 0)
       (effects (font (size 1.27 1.27)) hide)
     )
@@
     (property "Reference" "J2" (id 0) (at 112.776 148.59 0))
     (property "Value" "USB_A" (id 1) (at 112.776 151.13 0))
-    (property "Footprint" "easyeda2kicad:USB-A-SMD_USB-302S" (id 2) (at 112.776 153.67 0)
+    (property "Footprint" "easyeda2kicad:USB-A-SMD_GT-USB-2004-CWG1A" (id 2) (at 112.776 153.67 0)
       (effects (font (size 1.27 1.27)) hide)
     )
@@
       (effects (font (size 1.27 1.27)) hide)
     )
-    (property "LCSC" "C112455" (id 4) (at 112.776 164.084 0)
+    (property "LCSC" "C5117890" (id 4) (at 112.776 164.084 0)
       (effects (font (size 1.27 1.27)) hide)
     )
@@
       (reference "#PWR022") (unit 1) (value "+5V") (footprint "")
     )
+    (path "/05bf0b36-6e07-46d7-b7bd-213a32c3ae8d"
+      (reference "#PWR0101") (unit 1) (value "GND") (footprint "")
+    )
     (path "/89283c51-b7ea-4c70-8582-4ad0e5412d0a"
       (reference "#PWR0104") (unit 1) (value "GND") (footprint "")
@@
       (reference "#PWR0143") (unit 1) (value "GND") (footprint "")
     )
-    (path "/05bf0b36-6e07-46d7-b7bd-213a32c3ae8d"
-      (reference "#PWR?") (unit 1) (value "GND") (footprint "")
-    )
     (path "/351874dc-99f1-41fb-8357-28151f7d437e"
       (reference "C1") (unit 1) (value "100nF") (footprint "C_0402_1005Metric")
@@
     )
     (path "/bebad199-b672-4a4f-be0b-205c80aa969d"
-      (reference "J2") (unit 1) (value "USB_A") (footprint "easyeda2kicad:USB-A-SMD_USB-302S")
+      (reference "J2") (unit 1) (value "USB_A") (footprint "easyeda2kicad:USB-A-SMD_GT-USB-2004-CWG1A")
     )
     (path "/27715874-6fe4-4f69-aef5-1bdde490b73f"

Commit message: update schematic title
Other:
- title: MiSTeX Allwinner D1 cape for Terasic DECA -> MiSTeX Allwinner D1 Pmod
Changed lines of the file:
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@@
   (paper "A4")
   (title_block
-    (title "MiSTeX Allwinner D1 cape for Terasic DECA")
-    (date "2023-03-02")
+    (title "MiSTeX Allwinner D1 Pmod")
+    (date "2023-04-15")
     (rev "rev0")
     (company "Hans Baier")
