File: QMTech-MiSTeX/UserInterface.kicad_sch (KiCad schematic)
At the start: 84 parts, among them CN1 PJ-325C5-BL, CN2 U.FL-R-SMT-1(80), CN3 U.FL-R-SMT-1(80), CN4 U.FL-R-SMT-1(80), CN5 U.FL-R-SMT-1(80), J15 Conn_01x02_Pin, J16 Conn_01x02_Pin, J17 Conn_01x02_Pin, J19 Conn_01x02_Pin, J20 Conn_01x02_Pin, J21 Conn_01x02_Pin, J8 Conn_01x02_Pin, SW1 TS-1187A-B-A-B, SW2 TS-1187A-B-A-B, SW3 TS-1187A-B-A-B, SW4 TS-1187A-B-A-B, SW5 XKB5858-W-F-75, SW6 XKB5858-W-F-75, SW7 DSHP04TSGER, U5 ZGY133/T10(PLT)

Commit message: add rp2040 vbus, bump rev date, add USB_BOOT connection to RPi
Parts:
- J15, J16, J19, J20, J21, J8, TP10, TP11: now left out of the parts list
Changed lines of the file:
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@@
 		(unit 1)
 		(exclude_from_sim no)
-		(in_bom yes)
+		(in_bom no)
 		(on_board yes)
 		(dnp no)
@@
 		(unit 1)
 		(exclude_from_sim no)
-		(in_bom yes)
+		(in_bom no)
 		(on_board yes)
 		(dnp no)
@@
 		(unit 1)
 		(exclude_from_sim no)
-		(in_bom yes)
+		(in_bom no)
 		(on_board yes)
 		(dnp no)
@@
 		(unit 1)
 		(exclude_from_sim no)
-		(in_bom yes)
+		(in_bom no)
 		(on_board yes)
 		(dnp no)
@@
 		(unit 1)
 		(exclude_from_sim no)
-		(in_bom yes)
+		(in_bom no)
 		(on_board yes)
 		(dnp no)
@@
 		(unit 1)
 		(exclude_from_sim no)
-		(in_bom yes)
+		(in_bom no)
 		(on_board yes)
 		(dnp no)
@@
 		(unit 1)
 		(exclude_from_sim no)
-		(in_bom yes)
+		(in_bom no)
 		(on_board yes)
 		(dnp no)
@@
 		(unit 1)
 		(exclude_from_sim no)
-		(in_bom yes)
+		(in_bom no)
 		(on_board yes)
 		(dnp no)
