File: QMTech-MiSTeX/VGA.kicad_sch (KiCad schematic)
At the start: 19 parts, among them CN6 U.FL-R-SMT-1(80), CN7 U.FL-R-SMT-1(80), CN8 U.FL-R-SMT-1(80), J10 Conn_01x02

Commit message: add rp2040 vbus, bump rev date, add USB_BOOT connection to RPi
Parts:
- J10: now left out of the parts list
Changed lines of the file:
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@@
 		(unit 1)
 		(exclude_from_sim no)
-		(in_bom yes)
+		(in_bom no)
 		(on_board yes)
 		(dnp no)
